File: ergo42/ergo42.sch (KiCad schematic (older format))
At the start: 67 parts, among them J1 5PIN, SW1 SW_PUSH, SW10 SW_PUSH, SW11 SW_PUSH, SW12 SW_PUSH, SW13 SW_PUSH, SW14 SW_PUSH, SW15 SW_PUSH, SW16 SW_PUSH, SW17 SW_PUSH, SW18 SW_PUSH, SW19 SW_PUSH, SW2 SW_PUSH, SW20 SW_PUSH, SW21 SW_PUSH, SW22 SW_PUSH, SW23 SW_PUSH, SW24 SW_PUSH, SW25 SW_PUSH, SW26 SW_PUSH, SW27 SW_PUSH, SW28 SW_PUSH, SW29 SW_Push, SW3 SW_PUSH, SW4 SW_PUSH, SW5 SW_PUSH, SW6 SW_PUSH, SW7 SW_PUSH, SW8 SW_PUSH, SW9 SW_PUSH, U1 HOLE, U2 HOLE, U3 ProMicro, U4 HOLE, U5 HOLE, U7 HOLE

Commit message: Make meishi switch
Parts:
- removed D10, D11, D12, D14, D15, D16, D17, D18, D19, D2, D20, D21, D22, D23, D24, D25, D26, D27, D28, D3, D4, D6, D7, D8: D, library:Diode_SMD_THT, symbol D
- removed J1: 5PIN, library:trrs_jack, symbol 5PIN
- removed R1, R2: R, Resistors_THT:R_Axial_DIN0207_L6.3mm_D2.5mm_P10.16mm_Horizontal, symbol R
- removed SW10, SW11, SW12, SW14, SW15, SW16, SW17, SW18, SW19, SW2, SW20, SW21, SW22, SW23, SW24, SW25, SW26, SW27, SW28, SW3, SW4, SW6, SW7, SW8: SW_PUSH, library:key_switch, symbol SW_PUSH
- removed U1, U2, U4, U5, U7: HOLE, library:hole, symbol HOLE
- removed W1: jumper_smd, library:jumper_smd_2dub, symbol jumper_smd
Connections:
- net labels removed: col4, col5, col6, row1, row2, row3, scl, sda/uart, xtradata
- wire segments 39 -> 14
- no-connect marks 6 -> 14
